File: hardware/wisenode_v1.0.brd (EAGLE design)
At the start: 50 x 50 mm, 36 parts, among them J1 AUDIO-JACK2PTH, J2 M04X2, Q1 G2XX3---PW20, Q4 32.768 kHz, U1 MIC5025-3.3, X1 USBSMD

Commit message: changed LEDs, added push button
Parts:
- removed I/O, IRQ: (no value), led:CHIPLED_0805
- removed Q2: (no value), transistor:SOT23-BEC
- removed Q3: (no value), transistor-neu-to92:SOT23-BEC
- removed R4: 10K, resistor:M0805
- removed X1: USBSMD, SparkFun:USB-MINIB
- added RX: ORANGE, led:CHIPLED_0805
- added SW1: (no value), dp_devices:SW_TACT_SMALL
- added TX: GREEN, led:CHIPLED_0805
- added USB1: CON-USB-F-MINI-B, dp_devices:CONN_USB_MINI-B
- R1, R2: value 1K -> 220R
- moved R1 15.1 mm to (17.6, 1.57)
- moved R2 9.40 mm to (17.6, 4.24)
- moved R3 8.02 mm to (10.0, 3.05), turned to 90 degrees
- moved C5 4.76 mm to (20.8, 4.83), turned to 90 degrees
- moved R6 4.51 mm to (24.1, 1.65), turned to 180 degrees
- moved R9 0.40 mm to (16.9, 7.87)
- moved R10 0.36 mm to (17.9, 11.2)
- moved R8 0.18 mm to (16.9, 14.5)
- moved R5 0.13 mm to (13.6, 15.2)
Connections:
- net N$14 renamed TXD
- net N$5 renamed RST
- net N$9 renamed TST
- net P24 renamed RXD
- removed net N$10: Q3.B, R4.1
- removed net N$4: C3.1, Q1.19, Q4.1
- removed net N$6: I/O.C, Q2.C
- removed net N$7: Q2.B, R3.1
- removed net N$8: Q3.C, R2.1
- removed net P2.3: JP1.3, Q1.11
- removed net P2.4: JP1.2, Q1.12
- removed net P2.5: JP1.1, Q1.13
- new net BUTTON: JP1.1, Q1.13, R3.1, SW1.3, SW1.4
- new net N$5: Q1.12, R1.1
- new net P2.6: C3.1, JP1.2, Q1.19, Q4.1
- new net P2.7: C4.1, JP1.3, Q1.18, Q4.2
- net +3V3: now also RX.A, SW1.1, SW1.2, TX.A; no longer Q3.E, R1.1
- net GND: now also R3.2; no longer IRQ.C, Q2.E
- net IRQ: no longer R4.2
- net N$1: now also R2.2, TX.C; no longer I/O.A, R1.2
- net N$11: now also USB1.GND; no longer X1.GND
- net N$12: now also USB1.VUSB; no longer X1.VBUS
- net N$2: now also R1.2, RX.C; no longer IRQ.A, R2.2
- net N$3: now also Q1.11, R2.1; no longer C4.1, Q1.18, Q4.2
- net SCLK: no longer R3.2
Routing:
- net BUTTON: track 0.00 -> 58.3 mm, vias 0 -> 3
- net N$5: track 0.00 -> 23.5 mm, vias 0 -> 2
- net P2.7: track 0.00 -> 21.1 mm, vias 0 -> 1
- net P2.3: track 20.4 -> 0.00 mm, vias 2 -> 0
- net P2.6: track 0.00 -> 19.9 mm, vias 0 -> 1
- net P2.4: track 17.8 -> 0.00 mm, vias 2 -> 0
- net SCLK: track 36.1 -> 19.7 mm
- net N$4: track 15.2 -> 0.00 mm, vias 1 -> 0
- net P2.5: track 15.2 -> 0.00 mm, vias 2 -> 0
- net IRQ: track 29.4 -> 17.0 mm, vias 2 -> 1
- net N$6: track 10.1 -> 0.00 mm
- net N$3: track 13.5 -> 23.5 mm, vias 1 -> 2
- net +3V3: track 130.4 -> 138.9 mm
- net GND: track 136.1 -> 129.3 mm, vias 35 -> 33
- net RST: track 34.9 -> 39.0 mm
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Other:
- board text added: "BTN"
- board text added: "Magic Smoke"
- board text added: "P26"
- board text added: "P27"
- board text removed: "P23"
- board text removed: "P24"
- board text removed: "P25"
